Commit message: Gave up, creating new map

File: src/differential_drive_description/description/urdfs/bot.urdf (robot description, URDF)
Before this commit: robot differential_bot, 4 links, 3 joints
Joints:
- joint base_link_to_body: axis 1 0 0 -> (none); limit lower=-1.0 upper=1.0 effort=100 velocity=100 -> (none); origin xyz=0 0 ${body_z/2 + wheel_r} rpy=0 0 0 -> xyz=0.15 0 ${body_z/2 + wheel_r} rpy=0 0 0
